File: tdr.X/tdr.brd (EAGLE design)
At the start: 54.6 x 54.3 mm, 17 parts, among them IC1 PIC18F25K22-I_SP, X1 22-23-2021

Commit message: up
Parts:
- added SV4: (no value), con-lstb:MA04-1
- moved SV2 23.9 mm to (132.1, 27.9), turned to 0 degrees
- moved C3 8.89 mm to (151.1, 34.3)
- moved C2 6.35 mm to (151.1, 40.6)
- moved SV1 2.54 mm to (156.2, 67.3)
Connections:
- net CTPLS: now also SV4.1, SV4.2, SV4.3, SV4.4
Routing:
- net VSS: track 48.5 -> 29.8 mm, vias 0 -> 1
- net VDD: track 113.5 -> 128.4 mm
- net CTPLS: track 25.9 -> 36.2 mm
- net RX1: track 28.0 -> 19.3 mm
- net CTED1: track 31.1 -> 26.4 mm, vias 0 -> 1
- net TX1: track 28.0 -> 23.6 mm
- net CTED2: track 26.3 -> 27.4 mm
- net MCLR: track 31.0 -> 29.8 mm
- net PGC: track 14.7 -> 15.6 mm
