File: tdr.X/tdr.sch (EAGLE design)
At the start: 17 parts, among them IC1 PIC18F25K22-I_SP, X1 22-23-2021

Commit message: up
Parts:
- added SV4: (no value), con-lstb:MA04-1
Connections:
- net CTPLS: now also SV4.1, SV4.2, SV4.3, SV4.4
Changed lines of the file:
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@@
 <class number="0" name="default" width="0" drill="0">
+</class>
+<class number="1" name="icurrent" width="0.3048" drill="0">
 </class>
 </classes>
@@
 <part name="C4" library="rcl" library_urn="urn:adsk.eagle:library:334" deviceset="C-US" device="C0805" package3d_urn="urn:adsk.eagle:package:23617/2" value="0.1uf"/>
 <part name="VSS14" library="supply1" library_urn="urn:adsk.eagle:library:371" deviceset="VSS" device=""/>
+<part name="SV4" library="con-lstb" library_urn="urn:adsk.eagle:library:162" deviceset="MA04-1" device="" package3d_urn="urn:adsk.eagle:package:8337/1"/>
 </parts>
 <sheets>
@@
 <attribute name="VALUE" x="99.06" y="33.02" size="1.778" layer="96" rot="R270"/>
 </instance>
+<instance part="SV4" gate="1" x="134.62" y="83.82" smashed="yes">
+<attribute name="VALUE" x="133.35" y="73.66" size="1.778" layer="96"/>
+<attribute name="NAME" x="133.35" y="89.662" size="1.778" layer="95"/>
+</instance>
 </instances>
 <busses>
 </busses>
 <nets>
-<net name="CTED1" class="0">
+<net name="CTED1" class="1">
 <segment>
 <pinref part="IC1" gate="G$1" pin="RB2"/>
@@
 </segment>
 </net>
-<net name="CTED2" class="0">
+<net name="CTED2" class="1">
 <segment>
 <pinref part="IC1" gate="G$1" pin="RB3"/>
@@
 </segment>
 </net>
-<net name="VDD" class="0">
+<net name="VDD" class="1">
 <segment>
 <pinref part="C2" gate="G$1" pin="1"/>
@@
 </segment>
 </net>
-<net name="VSS" class="0">
+<net name="VSS" class="1">
 <segment>
 <pinref part="C1" gate="G$1" pin="2"/>
@@
 </segment>
 </net>
-<net name="CTPLS" class="0">
+<net name="CTPLS" class="1">
 <segment>
 <pinref part="IC1" gate="G$1" pin="RC2"/>
@@
 <junction x="154.94" y="53.34"/>
 </segment>
-</net>
+<segment>
+<wire x1="154.94" y1="78.74" x2="142.24" y2="78.74" width="0.1524" layer="91"/>
+<pinref part="SV4" gate="1" pin="1"/>
+<junction x="142.24" y="78.74"/>
+<junction x="154.94" y="78.74"/>
+<label x="147.32" y="78.74" size="1.778" layer="95"/>
+</segment>
+<segment>
+<wire x1="154.94" y1="81.28" x2="142.24" y2="81.28" width="0.1524" layer="91"/>
+<pinref part="SV4" gate="1" pin="2"/>
+<junction x="142.24" y="81.28"/>
+<junction x="154.94" y="81.28"/>
+<label x="147.32" y="81.28" size="1.778" layer="95"/>
+</segment>
+<segment>
+<wire x1="154.94" y1="83.82" x2="142.24" y2="83.82" width="0.1524" layer="91"/>
+<pinref part="SV4" gate="1" pin="3"/>
+<junction x="142.24" y="83.82"/>
+<junction x="154.94" y="83.82"/>
+<label x="147.32" y="83.82" size="1.778" layer="95"/>
+</segment>
+<segment>
+<wire x1="154.94" y1="86.36" x2="142.24" y2="86.36" width="0.1524" layer="91"/>
+<pinref part="SV4" gate="1" pin="4"/>
+<junction x="142.24" y="86.36"/>
+<junction x="154.94" y="86.36"/>
+<label x="147.32" y="86.36" size="1.778" layer="95"/>
+</segment>
+</net>

Commit message: up
Parts:
- added CTMU_ADC_PIN: TPB1,27, testpad:TPB1,27
- added TP1, TP2, TP3, TP4, TP5, TP6, TP7: TPPAD1-13, testpad:TPPAD1-13
Connections:
- new net N$3: CTMU_ADC_PIN.TP, IC1.RA0
- net CTED1: now also TP6.TP
- net CTED2: now also TP7.TP
- net CTPLS: now also TP2.TP
- net N$2: now also TP1.TP
- net N$4: now also TP3.TP
- net RX1: now also TP4.TP
- net TX1: now also TP5.TP
- net VDD: now also SV2.4
Changed lines of the file:
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@@
 <part name="VSS14" library="supply1" library_urn="urn:adsk.eagle:library:371" deviceset="VSS" device=""/>
 <part name="SV4" library="con-lstb" library_urn="urn:adsk.eagle:library:162" deviceset="MA04-1" device="" package3d_urn="urn:adsk.eagle:package:8337/1"/>
+<part name="CTMU_ADC_PIN" library="testpad" library_urn="urn:adsk.eagle:library:385" deviceset="TP" device="B1,27" package3d_urn="urn:adsk.eagle:package:27944/2"/>
+<part name="VDD8" library="supply1" library_urn="urn:adsk.eagle:library:371" deviceset="VDD" device=""/>
+<part name="TP1" library="testpad" library_urn="urn:adsk.eagle:library:385" deviceset="TP" device="PAD1-13" package3d_urn="urn:adsk.eagle:package:27946/1"/>
+<part name="TP2" library="testpad" library_urn="urn:adsk.eagle:library:385" deviceset="TP" device="PAD1-13" package3d_urn="urn:adsk.eagle:package:27946/1"/>
+<part name="TP3" library="testpad" library_urn="urn:adsk.eagle:library:385" deviceset="TP" device="PAD1-13" package3d_urn="urn:adsk.eagle:package:27946/1"/>
+<part name="TP4" library="testpad" library_urn="urn:adsk.eagle:library:385" deviceset="TP" device="PAD1-13" package3d_urn="urn:adsk.eagle:package:27946/1"/>
+<part name="TP5" library="testpad" library_urn="urn:adsk.eagle:library:385" deviceset="TP" device="PAD1-13" package3d_urn="urn:adsk.eagle:package:27946/1"/>
+<part name="TP6" library="testpad" library_urn="urn:adsk.eagle:library:385" deviceset="TP" device="PAD1-13" package3d_urn="urn:adsk.eagle:package:27946/1"/>
+<part name="TP7" library="testpad" library_urn="urn:adsk.eagle:library:385" deviceset="TP" device="PAD1-13" package3d_urn="urn:adsk.eagle:package:27946/1"/>
 </parts>
 <sheets>
@@
 <attribute name="NAME" x="133.35" y="89.662" size="1.778" layer="95"/>
 </instance>
+<instance part="CTMU_ADC_PIN" gate="G$1" x="38.1" y="60.96" smashed="yes" rot="R90">
+<attribute name="NAME" x="19.05" y="59.69" size="1.778" layer="95"/>
+<attribute name="TP_SIGNAL_NAME" x="39.37" y="62.23" size="1.778" layer="97" rot="R90"/>
+</instance>
+<instance part="VDD8" gate="G$1" x="96.52" y="15.24" smashed="yes" rot="R180">
+<attribute name="VALUE" x="99.06" y="17.78" size="1.778" layer="96" rot="R270"/>
+</instance>
+<instance part="TP1" gate="G$1" x="22.86" y="35.56" smashed="yes" rot="R90">
+<attribute name="NAME" x="21.59" y="34.29" size="1.778" layer="95" rot="R90"/>
+<attribute name="TP_SIGNAL_NAME" x="24.13" y="36.83" size="1.778" layer="97" rot="R90"/>
+</instance>
+<instance part="TP2" gate="G$1" x="30.48" y="33.02" smashed="yes" rot="R90">
+<attribute name="NAME" x="29.21" y="31.75" size="1.778" layer="95" rot="R90"/>
+<attribute name="TP_SIGNAL_NAME" x="31.75" y="34.29" size="1.778" layer="97" rot="R90"/>
+</instance>
+<instance part="TP3" gate="G$1" x="35.56" y="30.48" smashed="yes" rot="R90">
+<attribute name="NAME" x="34.29" y="29.21" size="1.778" layer="95" rot="R90"/>
+<attribute name="TP_SIGNAL_NAME" x="36.83" y="31.75" size="1.778" layer="97" rot="R90"/>
+</instance>
+<instance part="TP4" gate="G$1" x="83.82" y="20.32" smashed="yes" rot="R90">
+<attribute name="NAME" x="82.55" y="19.05" size="1.778" layer="95" rot="R90"/>
+<attribute name="TP_SIGNAL_NAME" x="85.09" y="21.59" size="1.778" layer="97" rot="R90"/>
+</instance>
+<instance part="TP5" gate="G$1" x="83.82" y="22.86" smashed="yes" rot="R90">
+<attribute name="NAME" x="82.55" y="21.59" size="1.778" layer="95" rot="R90"/>
+<attribute name="TP_SIGNAL_NAME" x="85.09" y="24.13" size="1.778" layer="97" rot="R90"/>
+</instance>
+<instance part="TP6" gate="G$1" x="96.52" y="48.26" smashed="yes" rot="R180">
+<attribute name="NAME" x="97.79" y="46.99" size="1.778" layer="95" rot="R180"/>
+<attribute name="TP_SIGNAL_NAME" x="95.25" y="49.53" size="1.778" layer="97" rot="R180"/>
+</instance>
+<instance part="TP7" gate="G$1" x="96.52" y="55.88" smashed="yes">
+<attribute name="NAME" x="95.25" y="57.15" size="1.778" layer="95"/>
+<attribute name="TP_SIGNAL_NAME" x="97.79" y="54.61" size="1.778" layer="97"/>
+</instance>
 </instances>
 <busses>
@@
 <segment>
 <pinref part="IC1" gate="G$1" pin="RB2"/>
-<wire x1="86.36" y1="50.8" x2="111.76" y2="50.8" width="0.1524" layer="91"/>
+<wire x1="86.36" y1="50.8" x2="96.52" y2="50.8" width="0.1524" layer="91"/>
 <label x="104.14" y="50.8" size="1.778" layer="95"/>
 <junction x="86.36" y="50.8"/>
 <junction x="111.76" y="50.8"/>
+<pinref part="TP6" gate="G$1" pin="TP"/>
+<wire x1="96.52" y1="50.8" x2="111.76" y2="50.8" width="0.1524" layer="91"/>
+<junction x="96.52" y="50.8"/>
 </segment>
 <segment>
@@
 <segment>
 <pinref part="IC1" gate="G$1" pin="RB3"/>
-<wire x1="86.36" y1="53.34" x2="111.76" y2="53.34" width="0.1524" layer="91"/>
+<wire x1="86.36" y1="53.34" x2="96.52" y2="53.34" width="0.1524" layer="91"/>
 <label x="104.14" y="53.34" size="1.778" layer="95"/>
 <junction x="86.36" y="53.34"/>
 <junction x="111.76" y="53.34"/>
+<pinref part="TP7" gate="G$1" pin="TP"/>
+<wire x1="96.52" y1="53.34" x2="111.76" y2="53.34" width="0.1524" layer="91"/>
+<junction x="96.52" y="53.34"/>
 </segment>
 <segment>
@@
 <pinref part="C4" gate="G$1" pin="1"/>
 <junction x="25.4" y="83.82"/>
+</segment>
+<segment>
+<pinref part="SV2" gate="1" pin="4"/>
+<pinref part="VDD8" gate="G$1" pin="VDD"/>
+<junction x="96.52" y="17.78"/>
 </segment>
 </net>
@@
 <junction x="96.52" y="22.86"/>
 <junction x="86.36" y="22.86"/>
+<pinref part="TP5" gate="G$1" pin="TP"/>
 </segment>
 </net>
@@
 <junction x="96.52" y="20.32"/>
 <junction x="86.36" y="20.32"/>
+<pinref part="TP4" gate="G$1" pin="TP"/>
 </segment>
 </net>
@@
 <pinref part="R3" gate="G$1" pin="2"/>
 <junction x="43.18" y="35.56"/>
+<pinref part="TP1" gate="G$1" pin="TP"/>
 <junction x="25.4" y="35.56"/>
 </segment>
@@
 <junction x="33.02" y="33.02"/>
 <label x="35.56" y="33.02" size="1.778" layer="95"/>
-</segment>
-<segment>
-<wire x1="111.76" y1="48.26" x2="101.6" y2="48.26" width="0.1524" layer="91"/>
+<pinref part="TP2" gate="G$1" pin="TP"/>
+</segment>
+<segment>
 <label x="104.14" y="48.26" size="1.778" layer="95"/>
 <junction x="101.6" y="48.26"/>
 <junction x="111.76" y="48.26"/>
+<wire x1="111.76" y1="48.26" x2="101.6" y2="48.26" width="0.1524" layer="91"/>
 </segment>
 <segment>
@@
 <junction x="43.18" y="30.48"/>
 <junction x="38.1" y="30.48"/>
+<pinref part="TP3" gate="G$1" pin="TP"/>
 </segment>
 </net>
@@
 </segment>
 </net>
+<net name="N$3" class="0">
+<segment>
+<pinref part="IC1" gate="G$1" pin="RA0"/>
+<pinref part="CTMU_ADC_PIN" gate="G$1" pin="TP"/>
+<wire x1="40.64" y1="60.96" x2="43.18" y2="60.96" width="0.1524" layer="91"/>
+<junction x="43.18" y="60.96"/>
+<junction x="40.64" y="60.96"/>
+</segment>
+</net>
