File: mate_a.sch (EAGLE design)
At the start: 8 parts, among them IC1 PIC18F47Q84-E_P, X1 GLX-S-88M

Commit message: up
Parts:
- removed IC1: PIC18F47Q84-E_P, PIC18F47Q84-E_P:PIC18F47Q84-E_P
- added 24VDC_PWR: 24vdc power, con-molex:22-23-2021
- added ANALOG: Analog, con-lstb:MA10-1
- added C1, C11, C12, C14, C16, C18, C2, C3, C5, C7, C9: 0.1uf, rcl:C-USC0805
- added C10, C13, C15, C17, C19, C4, C6, C8: 10uf, rcl:C-USC0805
- added CANBUS: CANBUS, con-lstb:MA04-1
- added CAN_PWR: CAN_PWR, jumper:SJ
- added DIGITAL: Digtal, con-lstb:MA10-1
- added EXT_IO: EXT_IO, con-lstb:MA06-1
- added IC2: 7805TV, linear:7805TV
- added IC3: ADM3095EBRZ, ADM3095EBRZ:ADM3095EBRZ
- added IC4: PIC18F47Q84-I_PT, PIC18F47Q84-I_PT:PIC18F47Q84-I_PT
- added ICSP: ICSP, con-lstb:MA06-1
- added LED1: run, led:LEDCHIPLED_0805
- added LED2: error, led:LEDCHIPLED_0805
- added LED3: comm, led:LEDCHIPLED_0805
- added MISC_IO: misc-io, con-lstb:MA10-1
- added MODBUS: MODBUS, pinhead:PINHD-1X5
- added OS1_10MHZ: OSC-OE-CFPS-72, IQD-Frequency-Products:OSC-OE-CFPS-72
- added R10: 120ohm, rcl:R-US_R0805
- added R11: 120, rcl:R-US_R0805
- added R12: 0 ohm fuse, rcl:R-US_R1206
- added R5: 56ohm, rcl:R-US_R0805
- added R6: 10k, rcl:R-US_R0805
- added R7, R8, R9: 1k, rcl:R-US_R0805
- added RESET: reset, jumper:SJ
- added R_RESET: remote_reset, pinhead:PINHD-1X2
- added TP1, TP2: PTR1PAD1-13, testpad:PTR1PAD1-13
- added TTL_SERIAL: TTL Serial, con-lstb:MA04-1
- added U1: REF3440IDBVR, REF3440IDBVR:REF3440IDBVR
- added U2: TCAN330GDR, TCAN330GDR:TCAN330GDR
- added VREF_PWR: 5vdc_vref_pwr, con-molex:22-23-2021
- added ZENER: 5.6V, diode:ZENER-DIODESMB
- R1, R2: value (none) -> 2.2k
- R3: value (none) -> 1k
- R4: value (none) -> 470ohm
- renumbered X1 to MATE
Connections:
- removed net PC_RX: IC1.RC7, OK1.EMI, R3.1
- removed net PC_TX: IC1.RC6, OK2.A
- new net AN0: ANALOG.10, IC4.RA0
- new net AN1: ANALOG.1, IC4.RA1
- new net AN2: ANALOG.2, IC4.RA2
- new net AN4: ANALOG.4, IC4.RA4
- new net AN5: ANALOG.5, IC4.RA5
- new net CANRX: IC4.RB0, U2.RXD
- new net CANTX: IC4.RB4, U2.TXD
- new net CAN_N: CANBUS.1, R10.1, U2.CANL
- new net CAN_P: CANBUS.3, R10.2, U2.CANH
- new net CAN_VCC: C7.1, C8.1, CANBUS.4, CAN_PWR.1, U2.VCC
- new net CLOCKO: IC4.RA6, MISC_IO.10
- new net CPU_CLK: IC4.RA7, OS1_10MHZ.OUT, TP2.TP
- new net CS: DIGITAL.3, IC4.RD3
- new net DB0: DIGITAL.1, IC4.RD1
- new net DB1: DIGITAL.2, IC4.RD2
- new net DERE: IC3.!RE, IC3.DE, IC4.RC2, TP1.TP
- new net DLED: IC4.RB3, IC4.RD4, MISC_IO.4, R9.2
- new net MB_A: IC3.A, MODBUS.3, R11.1
- new net MB_B: IC3.B, MODBUS.2, R11.2
- new net MB_RX: ANALOG.6, IC3.RXD, IC4.RC0
- new net MB_TX: ANALOG.7, IC3.TXD, IC4.RC1
- new net MCLR_SIG: IC4.VPP/!MCLR!/RE3, ICSP.1, MISC_IO.8, R5.2
- new net MISC: IC4.RE1, MISC_IO.2
- new net MLED: IC4.RB1, R7.2
- new net N$2: C14.1, C15.1, IC2.VI, R12.1
- new net N$4: LED1.A, R7.1
- new net N$5: LED2.A, R8.1
- new net N$6: LED3.A, R9.1
- new net PC_RX2: IC4.RD0, TTL_SERIAL.3
- new net PC_TX2: IC4.RD6, TTL_SERIAL.2
- new net PGC: EXT_IO.5, IC4.ICSPCLK/RB6, ICSP.5
- new net PGD: EXT_IO.6, IC4.ICSPDAT/RB7, ICSP.4
- new net RB5: EXT_IO.4, IC4.RB5, MISC_IO.6
- new net RD5: EXT_IO.2, IC4.RD5, MISC_IO.5
- new net RD7: EXT_IO.3, IC4.RD7, MISC_IO.7
- new net RE2: IC4.RE2, MISC_IO.3
- new net RELAY: IC4.RE0, MISC_IO.1
- new net RLED: IC4.RB2, R8.2
- new net R_RESET: C1.1, R5.1, R6.1, RESET.1, R_RESET.2
- new net SCK1: DIGITAL.4, IC4.RC3
- new net SDI1: DIGITAL.5, IC4.RC4
- new net SDO1: DIGITAL.6, IC4.RC5
- new net UC_RX: DIGITAL.10, IC4.RC7, OK1.EMI, R3.1
- new net UC_TX: DIGITAL.7, IC4.RC6, OK2.A
- new net V+: 24VDC_PWR-1.S, R12.2
- new net VREF: ANALOG.3, C16.1, C17.1, IC4.RA3, U1.OUT_F, U1.OUT_S, VREF_PWR-1.S
- net VDD: now also ANALOG.8, C10.1, C11.1, C12.1, C13.1, C18.1, C19.1, C2.1, C3.1, C4.1, C5.1, C6.1, C9.1, CAN_PWR.2, DIGITAL.8, IC2.VO, IC3.VCC, IC3.VIO, IC4.VDD_1, IC4.VDD_2, ICSP.2, MODBUS.5, OS1_10MHZ.CON, OS1_10MHZ.VDD, R6.2, TTL_SERIAL.4, U1.IN, ZENER.C; no longer IC1.VDD_1, IC1.VDD_2
- net VSS: now also 24VDC_PWR-2.S, ANALOG.9, C1.2, C10.2, C11.2, C12.2, C13.2, C14.2, C15.2, C16.2, C17.2, C18.2, C19.2, C2.2, C3.2, C4.2, C5.2, C6.2, C7.2, C8.2, C9.2, CANBUS.2, DIGITAL.9, EXT_IO.1, IC2.GND, IC3.GND_1, IC3.GND_2, IC3.GND_3, IC3.GND_4, IC3.GND_5, IC3.GND_6, IC3.GND_7, IC3.GND_8, IC4.VSS_1, IC4.VSS_2, ICSP.3, LED1.C, LED2.C, LED3.C, MISC_IO.9, MODBUS.1, MODBUS.4, OS1_10MHZ.VSS, RESET.2, R_RESET.1, TTL_SERIAL.1, U1.ENABLE, U1.GND_F, U1.GND_S, U2.GND, U2.S, U2.SHDN, VREF_PWR-2.S, ZENER.A; no longer IC1.VSS_1, IC1.VSS_2
