File: mate_a.sch (EAGLE design)
At the start: 59 parts, among them IC2 7805TV, IC3 ADM3095EBRZ, IC4 PIC18F47Q84-I_PT, U1 REF3440IDBVR, U2 TCAN330GDR

Commit message: up
Connections:
- net RD5 renamed AUX_RELAY
Other:
- note added: "blue"
- note added: "yellow"
Changed lines of the file:
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@@
 <sheet>
 <plain>
+<text x="10.16" y="0" size="1.778" layer="91">yellow</text>
+<text x="243.84" y="43.18" size="1.778" layer="91">blue</text>
 </plain>
 <instances>
@@
 </segment>
 </net>
-<net name="RD5" class="0">
+<net name="AUX_RELAY" class="0">
 <segment>
 <wire x1="86.36" y1="35.56" x2="111.76" y2="35.56" width="0.1524" layer="91"/>
